Commit message: test

File: src/articubot_one/description/gazebo_control.xacro (robot description, xacro)
@@ -42,6 +42,3 @@
         </joint>
     </ros2_control>
-    <gazebo>
-        <plugin name="gazebo_link_attacher" filename="libgazebo_link_attacher.so"/>
-    </gazebo>
 </robot>

File: src/articubot_one/description/robot_core.xacro (robot description, xacro)
@@ -39,5 +39,5 @@
         </geometry>
     </collision>
-    <xacro:inertial_box mass="20" x="0.3" y="0.3" z="0.15">
+    <xacro:inertial_box mass="50" x="0.3" y="0.3" z="0.15">
         <origin xyz="0 0 0.075" rpy="0 0 0"/>
     </xacro:inertial_box>
@@ -174,5 +174,5 @@
         </geometry>
     </collision>
-    <xacro:inertial_box mass="0.5" x="0.05" y="0.05" z="0.3">
+    <xacro:inertial_box mass="5" x="0.05" y="0.05" z="0.3">
         <origin xyz="0 0 0.15" rpy="0 0 0"/>
     </xacro:inertial_box>
@@ -184,4 +184,5 @@
     <axis xyz="0 0 1"/>
     <limit lower="0" upper="0.2" effort="1000" velocity="1.0"/>
+    <dynamics damping="50.0" friction="20.0"/>
 </joint>
 <link name="arm_base2">
@@ -199,5 +200,5 @@
         </geometry>
     </collision>
-    <xacro:inertial_box mass="0.2" x="0.05" y="0.54" z="0.05">
+    <xacro:inertial_box mass="5" x="0.05" y="0.54" z="0.05">
         <origin xyz="0 0 0" rpy="0 0 0"/>
     </xacro:inertial_box>
@@ -210,4 +211,5 @@
     <axis xyz="0 1 0"/>
     <limit lower="0" upper="0.26375" effort="1000" velocity="1.0"/>
+    <dynamics damping="50.0" friction="20.0"/>
 </joint>
 <link name="arm_link_L">
@@ -222,8 +224,8 @@
         <origin xyz="0.075 0 0" rpy="0 0 0"/>
         <geometry>
-            <box size="0.15 0.0125 0.05"/>
-        </geometry>
-    </collision>
-    <xacro:inertial_box mass="0.1" x="0.15" y="0.0125" z="0.05">
+            <box size="0.12 0.005 0.04"/>
+        </geometry>
+    </collision>
+    <xacro:inertial_box mass="2" x="0.15" y="0.0125" z="0.05">
         <origin xyz="0.075 0 0" rpy="0 0 0"/>
     </xacro:inertial_box>
@@ -243,4 +245,5 @@
     <axis xyz="0 1 0"/>
     <limit lower="-0.26375" upper="0" effort="1000" velocity="1.0"/>
+    <dynamics damping="50.0" friction="20.0"/>
 </joint>
 <link name="arm_link_R">
@@ -255,8 +258,8 @@
         <origin xyz="0.075 0 0" rpy="0 0 0"/>
         <geometry>
-            <box size="0.15 0.0125 0.05"/>
-        </geometry>
-    </collision>
-    <xacro:inertial_box mass="0.1" x="0.15" y="0.0125" z="0.05">
+            <box size="0.12 0.005 0.04"/>
+        </geometry>
+    </collision>
+    <xacro:inertial_box mass="2" x="0.15" y="0.0125" z="0.05">
         <origin xyz="0.075 0 0" rpy="0 0 0"/>
     </xacro:inertial_box>
@@ -269,10 +272,3 @@
         <material>Gazebo/White</material>
 </gazebo>
-<gazebo>
-  <plugin name="ifra_link_attacher_plugin" filename="libifra_link_attacher_plugin.so">
-    <ros>
-      <namespace>/</namespace>
-    </ros>
-  </plugin>
-</gazebo>
 </robot>
