Commit message: Add files via upload

File: src/articubot_one/description/robot_core.xacro (robot description, xacro)
@@ -39,6 +39,6 @@
         </geometry>
     </collision>
-    <xacro:inertial_box mass="50" x="0.3" y="0.3" z="0.15">
-        <origin xyz="0 0 0.075" rpy="0 0 0"/>
+    <xacro:inertial_box mass="200" x="0.3" y="0.3" z="0.15">
+        <origin xyz="-0.15 0 0.01" rpy="0 0 0"/>
     </xacro:inertial_box>
 </link>
@@ -50,5 +50,5 @@
     <parent link="base_link"/>
     <child link="front_left_wheel"/>
-    <origin xyz="0.075 0.17 0.05" rpy="-${pi/2} 0 0"/>
+    <origin xyz="0.14 0.17 0.05" rpy="-${pi/2} 0 0"/>
     <axis xyz="0 0 1"/>
 </joint>
@@ -73,5 +73,5 @@
     <parent link="base_link"/>
     <child link="back_left_wheel"/>
-    <origin xyz="-0.075 0.17 0.05" rpy="-${pi/2} 0 0"/>
+    <origin xyz="-0.14 0.17 0.05" rpy="-${pi/2} 0 0"/>
     <axis xyz="0 0 1"/>
 </joint>
@@ -96,5 +96,5 @@
     <parent link="base_link"/>
     <child link="front_right_wheel"/>
-    <origin xyz="0.075 -0.17 0.05" rpy="${pi/2} 0 0"/>
+    <origin xyz="0.14 -0.17 0.05" rpy="${pi/2} 0 0"/>
     <axis xyz="0 0 -1"/>
 </joint>
@@ -119,5 +119,5 @@
     <parent link="base_link"/>
     <child link="back_right_wheel"/>
-    <origin xyz="-0.075 -0.17 0.05" rpy="${pi/2} 0 0"/>
+    <origin xyz="-0.14 -0.17 0.05" rpy="${pi/2} 0 0"/>
     <axis xyz="0 0 -1"/>
 </joint>
@@ -183,5 +183,5 @@
     <origin xyz="0.05 0 0.025" rpy="0 0 0"/>
     <axis xyz="0 0 1"/>
-    <limit lower="0" upper="0.2" effort="1000" velocity="1.0"/>
+    <limit lower="0" upper="0.2" effort="1000" velocity="0.2"/>
     <dynamics damping="50.0" friction="20.0"/>
 </joint>
@@ -200,5 +200,5 @@
         </geometry>
     </collision>
-    <xacro:inertial_box mass="5" x="0.05" y="0.54" z="0.05">
+    <xacro:inertial_box mass="20" x="0.05" y="0.54" z="0.05">
         <origin xyz="0 0 0" rpy="0 0 0"/>
     </xacro:inertial_box>

Commit message: Add files via upload

File: src/articubot_one/description/robot_core.xacro (robot description, xacro)
@@ -39,6 +39,6 @@
         </geometry>
     </collision>
-    <xacro:inertial_box mass="200" x="0.3" y="0.3" z="0.15">
-        <origin xyz="-0.15 0 0.01" rpy="0 0 0"/>
+    <xacro:inertial_box mass="100" x="0.3" y="0.3" z="0.15">
+        <origin xyz="0 0 0.075" rpy="0 0 0"/>
     </xacro:inertial_box>
 </link>
@@ -50,5 +50,5 @@
     <parent link="base_link"/>
     <child link="front_left_wheel"/>
-    <origin xyz="0.14 0.17 0.05" rpy="-${pi/2} 0 0"/>
+    <origin xyz="0.075 0.17 0.05" rpy="-${pi/2} 0 0"/>
     <axis xyz="0 0 1"/>
 </joint>
@@ -73,5 +73,5 @@
     <parent link="base_link"/>
     <child link="back_left_wheel"/>
-    <origin xyz="-0.14 0.17 0.05" rpy="-${pi/2} 0 0"/>
+    <origin xyz="-0.075 0.17 0.05" rpy="-${pi/2} 0 0"/>
     <axis xyz="0 0 1"/>
 </joint>
@@ -96,5 +96,5 @@
     <parent link="base_link"/>
     <child link="front_right_wheel"/>
-    <origin xyz="0.14 -0.17 0.05" rpy="${pi/2} 0 0"/>
+    <origin xyz="0.075 -0.17 0.05" rpy="${pi/2} 0 0"/>
     <axis xyz="0 0 -1"/>
 </joint>
@@ -119,5 +119,5 @@
     <parent link="base_link"/>
     <child link="back_right_wheel"/>
-    <origin xyz="-0.14 -0.17 0.05" rpy="${pi/2} 0 0"/>
+    <origin xyz="-0.075 -0.17 0.05" rpy="${pi/2} 0 0"/>
     <axis xyz="0 0 -1"/>
 </joint>
